File: src/AQ_sensor/AQ_sensor_MRC.brd (EAGLE design)
At the start: 110 x 78 mm, 50 parts, among them IC2 MCP73831/OT, J1 F-1X03-SIP-100-32, SW1 PCM12SMTR, SW2 PCM12SMTR, U2 TEXAS_INSTRUMENTS_SN74HC125TE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, U3 TEXAS_INSTRUMENTS_LM1117IMP-3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, X1 53048-08, X2 SIMLOCK-C707_10M006_512_2, X4 50 Ohms

Commit message: Added Managed library to design
Parts:
- CN1: device AQ_sensor_WB_KE_KNBS:JST-PH-2-SMT-RA -> AQ_sensor_MRC:JST-PH-2-SMT-RA
- D1, D4, D5: device ON Semi - 1N4148WS:ON_SEMI_1N4148WS_0 -> AQ_sensor_MRC:ON_SEMI_1N4148WS_0
- D2: device On Semiconductor - MMSZ5231BT1G:ON_SEMICONDUCTOR_MMSZ5231BT1G_0 -> AQ_sensor_MRC:ON_SEMICONDUCTOR_MMSZ5231BT1G_0
- D3: device Semtech - SMF05C:SEMTECH_SMF05C_0 -> AQ_sensor_MRC:SEMTECH_SMF05C_0
- H1, H2, H3, H4: device AQ_sensor_WB_KE_KNBS:2,8-PAD -> AQ_sensor_MRC:2,8-PAD
- IC2: device adafruit:SOT23-5L -> AQ_sensor_MRC:SOT23-5L
- J1: device AQ_sensor_WB_KE_KNBS:SIP-100-03-32 -> AQ_sensor_MRC:SIP-100-03-32
- MICRO_USB: device AQ_sensor_WB_KE_KNBS:AMPHENOL_10118192-0001LF -> AQ_sensor_MRC:AMPHENOL_10118192-0001LF
- S1: device KMR621NGLFS:SW_KMR621NGLFS -> AQ_sensor_MRC:SW_KMR621NGLFS
- SV1, SV2: device AQ_sensor_WB_KE_KNBS:FE15 -> AQ_sensor_MRC:FE15
- SW1, SW2: device AQ_sensor_WB_KE_KNBS:SW_PCM12SMTR -> AQ_sensor_MRC:SW_PCM12SMTR
- U1: device adafruit:SIM800L -> AQ_sensor_MRC:SIM800L
- U2: device Texas Instruments - SN74HC125:TEXAS_INSTRUMENTS_SN74HC125_0 -> AQ_sensor_MRC:TEXAS_INSTRUMENTS_SN74HC125_0
- U3: device AQ_sensor_WB_KE_KNBS:TEXAS_INSTRUMENTS_LM1117IMP-3.3-NOPB_0 -> AQ_sensor_MRC:TEXAS_INSTRUMENTS_LM1117IMP-3.3-NOPB_0
- X1: device AQ_sensor_WB_KE_KNBS:53048-08 -> AQ_sensor_MRC:53048-08
- X2: device con-amphenol:C707_10M006_512_2 -> AQ_sensor_MRC:C707_10M006_512_2
- X4: device adafruit:SMA_EDGELAUNCH_UFL -> AQ_sensor_MRC:SMA_EDGELAUNCH_UFL

Commit message: Modifed RI LED connection
Connections:
- net +5V: now also R1.1; no longer RI.C
- net RI_5V: now also RI.C; no longer R1.1
Routing:
- net RI_5V: track 33.2 -> 36.7 mm, vias 3 -> 2
- net +5V: track 252.6 -> 251.7 mm, vias 10 -> 11
Changed lines of the file:
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@@
 <drawing>
 <settings>
-<setting alwaysvectorfont="yes"/>
+<setting alwaysvectorfont="no"/>
 <setting verticaltext="up"/>
 </settings>
@@
 <wire x1="108" y1="66.9" x2="108" y2="44.5" width="0.4" layer="1"/>
 <wire x1="106.925" y1="67.975" x2="108" y2="66.9" width="0.4" layer="1"/>
-<contactref element="RI" pad="C"/>
 <wire x1="15.4" y1="27.4" x2="12.1" y2="27.4" width="0.4" layer="16"/>
 <wire x1="12.1" y1="27.4" x2="11.9" y2="27.2" width="0.4" layer="16"/>
 <via x="11.9" y="27.2" extent="1-16" drill="0.35"/>
 <wire x1="11.9" y1="27.2" x2="10.9" y2="26.2" width="0.4" layer="1"/>
-<wire x1="2.1" y1="23" x2="2.1" y2="21.7" width="0.4" layer="1"/>
-<wire x1="2.1" y1="21.7" x2="3" y2="20.8" width="0.4" layer="1"/>
-<wire x1="5.25" y1="20.8" x2="5.35" y2="20.9" width="0.4" layer="1"/>
 <wire x1="10.9" y1="26.2" x2="5.3" y2="26.2" width="0.4" layer="1"/>
-<wire x1="5.3" y1="26.2" x2="2.1" y2="23" width="0.4" layer="1"/>
-<wire x1="3" y1="20.8" x2="5.25" y2="20.8" width="0.4" layer="1"/>
 <wire x1="14.2" y1="9.1" x2="13.7" y2="8.6" width="0.4" layer="1"/>
+<contactref element="R1" pad="1"/>
+<via x="5.3" y="26.2" extent="1-16" drill="0.35"/>
+<wire x1="5.3" y1="26.2" x2="4.1" y2="26.2" width="0.4" layer="16"/>
+<wire x1="2.2" y1="24.3" x2="2.2" y2="22.9" width="0.4" layer="16"/>
+<wire x1="2.2" y1="22.9" x2="3" y2="22.1" width="0.4" layer="16"/>
+<wire x1="3" y1="22.1" x2="5.15" y2="22.1" width="0.4" layer="16"/>
+<wire x1="4.1" y1="26.2" x2="2.2" y2="24.3" width="0.4" layer="16"/>
 </signal>
 <signal name="+3V3" class="1">
@@
 <signal name="RI_5V">
 <contactref element="U2" pad="11"/>
-<contactref element="R1" pad="1"/>
 <wire x1="15.825" y1="6.3" x2="17.5" y2="6.3" width="0.3" layer="1"/>
 <wire x1="17.5" y1="6.3" x2="18" y2="6.8" width="0.3" layer="1"/>
@@
 <wire x1="13.6" y1="22.9" x2="11.8" y2="24.7" width="0.3" layer="1"/>
 <wire x1="13.6" y1="18.6" x2="13.6" y2="22.9" width="0.3" layer="1"/>
-<via x="11.8" y="24.7" extent="1-16" drill="0.35"/>
-<wire x1="11.8" y1="24.7" x2="5.8" y2="24.7" width="0.3" layer="16"/>
-<wire x1="5.15" y1="24.05" x2="5.15" y2="22.1" width="0.3" layer="16"/>
-<wire x1="5.8" y1="24.7" x2="5.15" y2="24.05" width="0.3" layer="16"/>
+<contactref element="RI" pad="C"/>
+<wire x1="11.8" y1="24.7" x2="5.9" y2="24.7" width="0.3" layer="1"/>
+<wire x1="3.4" y1="21.3" x2="3.8" y2="20.9" width="0.3" layer="1"/>
+<wire x1="3.8" y1="20.9" x2="5.35" y2="20.9" width="0.3" layer="1"/>
+<wire x1="5.9" y1="24.7" x2="3.4" y2="22.2" width="0.3" layer="1"/>
+<wire x1="3.4" y1="22.2" x2="3.4" y2="21.3" width="0.3" layer="1"/>
 </signal>
 <signal name="N$14">

Commit message: Added ground vias
Routing:
- net GND: vias 3 -> 9
Changed lines of the file:
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@@
 <wire x1="28.368" y1="2.332" x2="27" y2="3.7" width="0.3" layer="1"/>
 <wire x1="31.46" y1="2.332" x2="31.46" y2="2.332" width="0" layer="19" extent="1-16"/>
+<via x="38.4" y="1" extent="1-16" drill="0.35"/>
+<via x="38.4" y="2.8" extent="1-16" drill="0.35"/>
+<via x="38.2" y="4.2" extent="1-16" drill="0.35"/>
+<via x="29" y="1.3" extent="1-16" drill="0.35"/>
+<via x="29.5" y="3.3" extent="1-16" drill="0.35"/>
+<via x="29.8" y="4.5" extent="1-16" drill="0.35"/>
 </signal>
 <signal name="+5V" class="1">
@@
 <wire x1="55.7" y1="27.9" x2="53.9" y2="26.1" width="0.3" layer="1"/>
 </signal>
-<signal name="N$1">
-<via x="29.8" y="4.5" extent="1-16" drill="0.35"/>
-</signal>
-<signal name="N$2">
-<via x="29.5" y="3.3" extent="1-16" drill="0.35"/>
-</signal>
-<signal name="N$3">
-<via x="29" y="1.3" extent="1-16" drill="0.35"/>
-</signal>
-<signal name="N$5">
-<via x="38.4" y="1" extent="1-16" drill="0.35"/>
-</signal>
-<signal name="N$7">
-<via x="38.4" y="2.8" extent="1-16" drill="0.35"/>
-</signal>
-<signal name="N$8">
-<via x="38.2" y="4.2" extent="1-16" drill="0.35"/>
-</signal>
 <signal name="RI_5V">
